File: hardware/kicad/generated/harman-kardom.kicad_sch (KiCad schematic)
At the start: 27 parts, among them J1 USB-C PD INPUT, J2 WOOFER / IMPEDANCE TBD, J3 TWEETER / IMPEDANCE TBD, SW1 FUNCTION / RESET / PROVISION, U1 USB-C PD TRIGGER / 20 V, U2 XL4015 CC/CV / 16.80 V 2.00 A, U3 4S BALANCED BMS / COMMON PORT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, U4 MP1584 / ADJUST TO 5.10 V, U5 ESP32-S3 N16R8 DEV BOARD, U6 PCM5102A I2S DAC MODULE, U7 XH-A232 / TPA3110 BTL AMP

Commit message: docs: align vault with ADR-0009/0010, rework schematics, stage firmware plan
Close the drift between the canonical plans and what was actually costed and
drawn, then make the drawings and the verification reproducible.

Decisions recorded
  ADR-0009  V1 charge chain: USB-C PD -> 20 V trigger -> XL4015 16.80 V/2.00 A
            CC/CV -> 4S BMS. The chain was already priced and drawn but never
            decided; the canonical power and wiring plans still described a
            plain 16.8 V brick. Records the open charge-termination risk: the
            XL4015 is a generic CC/CV buck with no termination guarantee, and
            the BMS overcharge cut-off is not a charge algorithm.
  ADR-0010  Board locked to ESP32-S3 N16R8. The OTA manifest, pin plan and both
            drawings still said N8R8, which contradicts ADR-0008's dual OTA
            slot budget.

Documentation integrity
  Add scripts/check_docs.py: wiki links, docs/ frontmatter, ADR status
  vocabulary, ADR index completeness, agent/skill schema, and drift from the
  locked decisions. Five development logs claimed a link check had been run
  while no such tool existed in the repository.
  Add G4 charge-chain measurement table, four risk-register rows, supersede
  pointers on two outdated cost logs, and missing owner fields.

Agent infrastructure
  Six roles now exist in all three tools: explorer, hardware-worker,
  firmware-worker, acoustics-worker, hardware-reviewer, verifier. Previously
  explorer lived only in Codex and the two writer roles did not exist, while
  the documentation drew all of them.

Firmware
  Rewrite the plan as staged F0-F8 with preconditions, measurable acceptance
  criteria and gate mapping. F1 (AirPlay feasibility spike) is placed before
  expensive hardware work.

Drawings
  Replace two overlapping hand-written SVGs and their PNGs with one generated
  sheet. Rewrite the KiCad generator with real symbols, a 2.54 mm grid, wire
  endpoints resolved from pin positions, drawn wi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
Parts:
- removed JTP1: TP0-TP9 POWER, symbol Connector_Generic:Conn_01x10
- removed JTP2: TP10-TP17 SIGNAL, symbol Connector_Generic:Conn_01x08
- removed JTP3: TP18-TP25 BTL/CHARGE, symbol Connector_Generic:Conn_01x08
- removed U5: ESP32-S3 N16R8 DEV BOARD, symbol Connector_Generic:Conn_01x16
- removed U6: PCM5102A I2S DAC MODULE, symbol Connector_Generic:Conn_01x12
- removed U7: XH-A232 / TPA3110 BTL AMP, symbol Connector_Generic:Conn_01x10
- added C3: C_DB / 100 nF HARDWARE DEBOUNCE / OPTIONAL, symbol Device:C
- added F2: F_CHG / 3 A CANDIDATE, symbol Device:Fuse
- added R3: R_R / 680 R CANDIDATE, symbol Device:R
- added R4: R_G / 330 R CANDIDATE, symbol Device:R
- added R5: R_B / 330 R CANDIDATE, symbol Device:R
- added TP0: BMINUS, symbol Connector:TestPoint
- added TP1: B1, symbol Connector:TestPoint
- added TP10: ESP_3V3, symbol Connector:TestPoint
- added TP11: I2S_BCLK, symbol Connector:TestPoint
- added TP12: I2S_LRCLK, symbol Connector:TestPoint
- added TP13: I2S_DATA, symbol Connector:TestPoint
- added TP14, TP16: DAC_LOUT, symbol Connector:TestPoint
- added TP15, TP17: DAC_ROUT, symbol Connector:TestPoint
- added TP18: AMP_L_PLUS, symbol Connector:TestPoint
- added TP19: AMP_L_MINUS, symbol Connector:TestPoint
- added TP2: B2, symbol Connector:TestPoint
- added TP20: AMP_R_PLUS, symbol Connector:TestPoint
- added TP21: AMP_R_MINUS, symbol Connector:TestPoint
- added TP22: BUTTON_N, symbol Connector:TestPoint
- added TP23: LED_R, symbol Connector:TestPoint
- added TP24: LED_G, symbol Connector:TestPoint
- added TP25: LED_B, symbol Connector:TestPoint
- added TP26: CHG_16V8, symbol Connector:TestPoint
- added TP27: NTC_BMS, symbol Connector:TestPoint
- added TP3: B3, symbol Connector:TestPoint
- added TP4: BPLUS, symbol Connector:TestPoint
- added TP5: PACK_POS, symbol Connector:TestPoint
- added TP6: POWER_GND, symbol Connector:TestPoint
- added TP7: FUSED_POS, symbol Connector:TestPoint
- added TP8: VBAT_SW, symbol Connector:TestPoint
- added TP9: V5_SYS, symbol Connector:TestPoint
- added U5: ESP32-S3 DEVKIT N16R8 / 16 MB FLASH + 8 MB PSRAM, symbol Connector_Generic:Conn_01x13
- added U6: PCM5102A I2S DAC MODULE / 3-WIRE PLL, symbol Connector_Generic:Conn_01x09
- added U7: XH-A232 TPA3110 BTL AMP / 8-26 V, symbol Connector_Generic:Conn_01x09
- BT1: value ASPILSAN A28 18650 / CELL 1 -> ASPILSAN INR18650A28 / CELL 4
- BT2: value ASPILSAN A28 18650 / CELL 2 -> ASPILSAN INR18650A28 / CELL 3
- BT3: value ASPILSAN A28 18650 / CELL 3 -> ASPILSAN INR18650A28 / CELL 2
- BT4: value ASPILSAN A28 18650 / CELL 4 -> ASPILSAN INR18650A28 / CELL 1
- C1: value 1000 uF / 25 V LOW-ESR -> 1000 uF / 25 V / 105 C LOW-ESR TARGET
- C2: value C_SAFE / TBD FILM HPF -> C_SAFE / NON-POLARISED FILM / VALUE TBD UNTIL G2
- D1: value COMMON-CATHODE RGB LED -> COMMON-CATHODE RGB STATUS LED
- D2: value KM103 INTERNAL 12 V LED -> KM103 INTERNAL 12 V LAMP / DNP
- J1: value USB-C PD INPUT -> USB-C PD INLET / EXTERNAL 65 W ADAPTER
- J2: value WOOFER / IMPEDANCE TBD -> WOOFER / IMPEDANCE TBD / G0
- J3: value TWEETER / IMPEDANCE TBD -> TWEETER / IMPEDANCE TBD / G2
- JP1: value USB-SYSTEM 5 V ISOLATION -> USB / SYSTEM 5 V ISOLATION JUMPER
- R1: value 10 k PULL-UP -> 10 k PULL-UP CANDIDATE
- R2: value R_SW_LED TBD / DNP -> R_SW_LED / VALUE TBD / DNP
- S1: value KM103 / DC-132A CONTACTS / VERIFY 16.8 VDC 5 A -> KM103 / DC-132A / CONTACT RATING UNDOCUMENTED / VERIFY 16.8 VDC 5 A
- SW1: value FUNCTION / RESET / PROVISION -> FUNCTION / PROVISION / RESET
- U1: value USB-C PD TRIGGER / 20 V -> USB-C PD TRIGGER / FIXED 20 V
- U2: value XL4015 CC/CV / 16.80 V 2.00 A -> XL4015 CC-CV / CALIBRATE 16.80 V 2.00 A
- U3: value 4S BALANCED BMS / COMMON PORT CANDIDATE -> 4S BALANCED BMS / COMMON PORT / VERIFY SILKSCREEN
- U4: value MP1584 / ADJUST TO 5.10 V -> MP1584 BUCK / SET 5.10 V UNLOADED
Connections:
- net BUTTON_N is gone; now on net STAR_GND: R1.2, SW1.2
- net CHG_NEG is gone; now on net POWER_GND: U2.4 (Pin_4)
- net ESP_3V3 is gone; now on net STAR_GND: R1.1
- net PACK_NEG is gone; now on net POWER_GND: U3.7 (Pin_7)
- net PACK_POS is gone; now on net FUSED_POS: F1.2, U3.6 (Pin_6)
- net TWEETER_POS is gone; now on net AMP_R_PLUS: C2.1, J3.1 (Pin_1)
- net AMP_L_MINUS: now also TP19.1, U7.6 (Pin_6)
- net AMP_L_PLUS: now also TP18.1, U7.5 (Pin_5)
- net AMP_MUTE_TBD: now also U5.13 (Pin_13)
- net AMP_R_MINUS: now also TP21.1, U7.8 (Pin_8)
- net AMP_R_PLUS: now also TP20.1, U7.7 (Pin_7)
- net AMP_SD_TBD: now also U7.9 (Pin_9)
- net B1: now also U3.4 (Pin_4), TP1.1; no longer U3.2 (Pin_2)
- net B2: now also TP2.1
- net B3: now also U3.2 (Pin_2), TP3.1; no longer U3.4 (Pin_4)
- net BMINUS: now also U3.5 (Pin_5), TP0.1; no longer U3.1 (Pin_1)
- net BPLUS: now also U3.1 (Pin_1), TP4.1; no longer U3.5 (Pin_5)
- net CHG_16V8: now also F2.2, TP26.1
- net DAC_AGND: now also U6.9 (Pin_9)
- net DAC_LOUT: now also TP14.1, TP16.1, U6.7 (Pin_7), U7.1 (Pin_1)
- net DAC_ROUT: now also TP15.1, TP17.1, U6.8 (Pin_8), U7.2 (Pin_2)
- net FUSED_POS: now also F2.1, TP5.1, TP7.1
- net I2C_SCL: now also U5.12 (Pin_12)
- net I2C_SDA: now also U5.11 (Pin_11)
- net I2S_BCLK: now also TP11.1, U5.8 (Pin_8), U6.1 (Pin_1)
- net I2S_DATA: now also TP13.1, U5.10 (Pin_10), U6.3 (Pin_3)
- net I2S_LRCLK: now also TP12.1, U5.9 (Pin_9), U6.2 (Pin_2)
- net LED_B: now also R5.2, TP25.1, U5.7 (Pin_7); no longer D1.3 (Pin_3)
- net LED_G: now also R4.2, TP24.1, U5.6 (Pin_6); no longer D1.2 (Pin_2)
- net LED_R: now also R3.2, TP23.1, U5.5 (Pin_5); no longer D1.1 (Pin_1)
- net NTC_BMS: now also TP27.1
- net POWER_GND: now also TP6.1, U7.4 (Pin_4)
- net STAR_GND: now also C3.1, C3.2, TP10.1, TP22.1, U5.2 (Pin_2), U5.3 (Pin_3), U5.4 (Pin_4), U6.4 (Pin_4), U6.6 (Pin_6)
- net V5_LOGIC: now also U5.1 (Pin_1), U6.5 (Pin_5)
- net V5_SYS: now also TP9.1
- net VBAT_SW: now also TP8.1, U7.3 (Pin_3)
- net SW_LED_RETURN_TBD renamed SW_LED_RETURN
- new net LED_B_A: D1.3 (Pin_3), R5.1
- new net LED_G_A: D1.2 (Pin_2), R4.1
- new net LED_R_A: D1.1 (Pin_1), R3.1
Other:
- note added: "A. USB-C PD INPUT AND 16.80 V CC-CV CHARGE STAGE (ADR-0009)"
- note added: "Adjust U4 to 5.10 V before connecting the ESP32 and DAC. Keep JP1 open while programming over USB."
- note added: "B. 4S PACK, BALANCED BMS, FUSE AND HARD POWER SWITCH"
- note added: "BMS pin order is logical. Verify silkscreen, real continuous current, balance threshold/current and NTC behaviour before wiring."
- note added: "Button, LED and I2C wiring is kept away from the Class-D speaker cables. GPIO assignment is a candidate until the board schematic and a boot test exist."
- note added: "C. 5 V LOGIC SUPPLY"
- note added: "C_SAFE is not a crossover. It is the last line of defence behind the DSP high-pass and limiter; its value comes from the G2 report."
- note added: "D. ESP32-S3 N16R8 AND USER INTERFACE (ADR-0010)"
- note added: "D2 and R2 stay DNP: the switch lamp is a 12 V part and is never connected directly to the 16.8 V rail."
- note added: "DANGER: AMP_L_MINUS and AMP_R_MINUS are BTL switching outputs, not ground. Never clip a scope ground to them."
- note added: "E. I2S DAC, BTL BI-AMP AND DRIVERS (ADR-0002)"
- note added: "F. TEST POINT ACCESS TP0-TP27"
- note added: "G0 driver impedance BLOCKED | G1 dummy-load amp BLOCKED | G2 tweeter HPF and C_SAFE BLOCKED | G3 power, ripple, EMI BLOCKED | G4 battery, charge termination, NTC BLOCKED"
- note added: "Left digital channel drives the woofer path, right drives the tweeter path. This is a bi-amp split of one mono program, not a stereo box."
- note added: "Module connectors show a logical interface, not a seller board's physical pin order. Confirm every silkscreen and datasheet before wiring hardware."
- note added: "Scope ground goes to POWER_GND or STAR_GND only. For BTL outputs use a differential probe, or two 10x probes with BOTH ground clips on TP6 and MATH = CH1 - CH2."
- note added: "Series resistors are DNP if the purchased RGB module already carries them."
- note added: "Set the PD trigger to 20 V and calibrate the XL4015 to 16.80 V / 2.00 A WITH THE BATTERY DISCONNECTED."
- note added: "TP9 target: <=50 mVpp under normal load; the 5 V rail must not dip below 4.75 V on Wi-Fi current bursts."
- note added: "XL4015 HAS NO GUARANTEED CHARGE TERMINATION. Measure the CV current decay at G4; no unattended charging before that."
- note removed: "A. USB-C PD + 4S CC/CV CHARGE"
- note removed: "Adjust U4 to 5.10 V before connecting ESP32/DAC. Keep JP1 open until USB backfeed safety is proven."
- note removed: "Avoid strapping GPIO0/3/45/46 and native USB GPIO19/20."
- note removed: "B. 4S PACK, BMS, FUSE, HARD POWER"
- note removed: "BMS pin order is logical only. Verify actual silkscreen, balance threshold/current and NTC behavior."
- note removed: "C. SWITCHED POWER"
- note removed: "C_SAFE remains TBD until tweeter DCR/impedance and safe HPF are measured."
- note removed: "Calibrate XL4015 to 16.80 V / 2.00 A on a dummy load. V1: CHARGE WHILE PLAYING DISABLED."
- note removed: "D. ESP32-S3 + USER INTERFACE"
- note removed: "DANGER: L-/R- are BTL switching outputs. NEVER connect them to GND."
- note removed: "E. I2S DAC + BTL AMP + DRIVERS"
- note removed: "F. TEST POINTS / OSCILLOSCOPE ACCESS"
- note removed: "G0 driver impedance BLOCKED | G1 dummy-load amp BLOCKED | G2 C_SAFE BLOCKED | G3 power/thermal BLOCKED | G4 battery/BMS BLOCKED"
- note removed: "GPIO candidates: BCLK=4, LRCLK=5, DATA=6, BTN=7, RGB=8/9/10, I2C=11/12."
- note removed: "PCM5102A: SCK->GND for 3-wire PLL; verify module solder bridges."
- note removed: "S1 contact rating is undocumented: verify 16.8 VDC / 5 A. D2 is 12 V only; keep R2 DNP until LED current is measured."
- note removed: "Scope ground: POWER_GND/STAR_GND only. For BTL use a differential probe or CH1-CH2; both ground clips at POWER_GND."
- note removed: "Set PD trigger to 20 V without the battery connected."
- title: Harman Kardom - Module-Level Prototype -> Harman Kardom - Single Speaker, Module Level
